File: Hardware/Main Board/Main Board.sch (KiCad schematic (older format))
At the start: 8 parts, among them Q1 NPN

Commit message: schemaic
Parts:
- removed TP1: OUTPUT, symbol Connector:TestPoint
- added C2, C3: 10uf, symbol Device:CP1_Small
- added C? (x2): ?uf, symbol Device:CP1_Small
- added Q2: NPN, symbol Device:Q_NPN_BEC
- added R5: 100k, symbol Device:R_Small
- added R6: 10k, symbol Device:R_Small
- added R7: 1k, symbol Device:R_Small
- added TP2: OUTPUT, symbol Connector:TestPoint
- R1: value 10k -> 6.8k
Connections:
- net +5V: now also R1.2, R6.1; no longer R1.1
- net GND: now also C?.2, C?.2, R7.2
- net at C1.1, MK1.2 (+): now also R1.1; no longer R1.2
- net at C1.2, Q1.1 (B): now also R2.1; no longer R2.2
- net at Q1.2 (E), R4.1: now also C?.1
- net at Q1.3 (C), R3.2: now also R2.2, C2.1; no longer R2.1
- new net: C2.2, Q2.1 (B), R5.1
- new net: C3.1, Q2.3 (C), R5.2, R6.2
- new net: C3.2, TP2.1
- new net: C?.1, Q2.2 (E), R7.1
Other:
- moved on the sheet: C1, MK1

Commit message: shcmeatic tuning
Parts:
- removed C?: ?uf, symbol Device:CP1_Small
- C4: renamed from C?; value ?uf -> 0.1uf
- R1: value 6.8k -> 10k
Changed lines of the file:
@@
 P 1790 2180
 F 0 "R1" H 1849 2226 50  0000 L CNN
-F 1 "6.8k" H 1849 2135 50  0000 L CNN
+F 1 "10k" H 1849 2135 50  0000 L CNN
 F 2 "" H 1790 2180 50  0001 C CNN
 F 3 "~" H 1790 2180 50  0001 C CNN
@@
 	2940 1670 2940 1930
 $Comp
-L Device:CP1_Small C?
-U 1 1 5EB5411B
-P 3510 2730
-F 0 "C?" H 3360 2740 50  0000 C CNN
-F 1 "?uf" H 3360 2650 50  0000 C CNN
-F 2 "" H 3510 2730 50  0001 C CNN
-F 3 "~" H 3510 2730 50  0001 C CNN
-	1    3510 2730
-	1    0    0    -1
-$EndComp
-Wire Wire Line
-	3510 2630 3710 2630
-Connection ~ 3710 2630
-Wire Wire Line
-	3510 2830 3710 2830
-Connection ~ 3710 2830
-$Comp
-L Device:CP1_Small C?
+L Device:CP1_Small C4
 U 1 1 5EB56011
 P 2800 2720
-F 0 "C?" H 2650 2760 50  0000 C CNN
-F 1 "?uf" H 2650 2670 50  0000 C CNN
+F 0 "C4" H 2650 2760 50  0000 C CNN
+F 1 "0.1uf" H 2620 2680 50  0000 C CNN
 F 2 "" H 2800 2720 50  0001 C CNN
 F 3 "~" H 2800 2720 50  0001 C CNN

Commit message: failed boost converter
Parts:
- added BT1: 3.8V, symbol Device:Battery_Cell
- added C5: C_Small, symbol Device:C_Small
- added D1: D_ALT, symbol Device:D_ALT
- added L1: L_Core_Iron, symbol Device:L_Core_Iron
- added Q3: A0448, Package_TO_SOT_SMD:TDSON-8-1, symbol Transistor_FET:CSD16342Q5A
- added TP1: 12V+, symbol Connector:TestPoint
- added TP3: 12V-, symbol Connector:TestPoint
Connections:
- wire segments 23 -> 34
Changed lines of the file:
@@
 EESchema Schematic File Version 4
+LIBS:Main Board-cache
 EELAYER 30 0
 EELAYER END
@@
 	2800 2620 2940 2620
 Connection ~ 2940 2620
+$Comp
+L Transistor_FET:CSD16342Q5A Q3
+U 1 1 5EBD05D1
+P 5340 2660
+F 0 "Q3" H 5130 2370 50  0000 L CNN
+F 1 "A0448" H 5130 2290 50  0000 L CNN
+F 2 "Package_TO_SOT_SMD:TDSON-8-1" H 5540 2585 50  0001 L CIN
+F 3 "http://www.ti.com/lit/gpn/csd16342q5a" V 5340 2660 50  0001 L CNN
+	1    5340 2660
+	1    0    0    -1
+$EndComp
+$Comp
+L Device:Battery_Cell BT1
+U 1 1 5EBF3FED
+P 4470 2710
+F 0 "BT1" H 4588 2806 50  0000 L CNN
+F 1 "3.8V" H 4588 2715 50  0000 L CNN
+F 2 "" V 4470 2770 50  0001 C CNN
+F 3 "~" V 4470 2770 50  0001 C CNN
+	1    4470 2710
+	1    0    0    -1
+$EndComp
+Wire Wire Line
+	4470 2860 5440 2860
+Wire Wire Line
+	4470 2460 4750 2460
+$Comp
+L Device:D_ALT D1
+U 1 1 5EBE76EE
+P 5590 2460
+F 0 "D1" H 5590 2244 50  0000 C CNN
+F 1 "D_ALT" H 5590 2335 50  0000 C CNN
+F 2 "" H 5590 2460 50  0001 C CNN
+F 3 "~" H 5590 2460 50  0001 C CNN
+	1    5590 2460
+	-1   0    0    1
+$EndComp
+Wire Wire Line
+	5050 2460 5440 2460
+$Comp
+L Device:L_Core_Iron L1
+U 1 1 5EBCB70E
+P 4900 2460
+F 0 "L1" V 4719 2460 50  0000 C CNN
+F 1 "L_Core_Iron" V 4810 2460 50  0000 C CNN
+F 2 "" H 4900 2460 50  0001 C CNN
+F 3 "~" H 4900 2460 50  0001 C CNN
+	1    4900 2460
+	0    1    1    0
+$EndComp
+$Comp
+L Device:C_Small C5
+U 1 1 5EBEE2F7
+P 5810 2680
+F 0 "C5" H 5902 2726 50  0000 L CNN
+F 1 "C_Small" H 5902 2635 50  0000 L CNN
+F 2 "" H 5810 2680 50  0001 C CNN
+F 3 "~" H 5810 2680 50  0001 C CNN
+	1    5810 2680
+	1    0    0    -1
+$EndComp
+Connection ~ 5440 2460
+Wire Wire Line
+	4470 2460 4470 2510
+Wire Wire Line
+	4470 2810 4470 2860
+Wire Wire Line
+	5440 2860 5810 2860
+Wire Wire Line
+	5810 2860 5810 2780
+Connection ~ 5440 2860
+Wire Wire Line
+	5740 2460 5810 2460
+Wire Wire Line
+	5810 2460 5810 2580
+Wire Wire Line
+	5810 2460 6480 2460
+Connection ~ 5810 2460
+Wire Wire Line
+	5810 2860 6480 2860
+Connection ~ 5810 2860
+$Comp
+L Connector:TestPoint TP1
+U 1 1 5EC32DDA
+P 6480 2460
+F 0 "TP1" V 6434 2648 50  0000 L CNN
+F 1 "12V+" V 6525 2648 50  0000 L CNN
+F 2 "" H 6680 2460 50  0001 C CNN
+F 3 "~" H 6680 2460 50  0001 C CNN
+	1    6480 2460
+	0    1    1    0
+$EndComp
+$Comp
+L Connector:TestPoint TP3
+U 1 1 5EC34CEF
+P 6480 2860
+F 0 "TP3" V 6434 3048 50  0000 L CNN
+F 1 "12V-" V 6525 3048 50  0000 L CNN
+F 2 "" H 6680 2860 50  0001 C CNN
+F 3 "~" H 6680 2860 50  0001 C CNN
+	1    6480 2860
+	0    1    1    0
+$EndComp
 $EndSCHEMATC

Commit message: added boost converter, button and ton of work to schematic
Parts:
- removed BT1: 3.8V, symbol Device:Battery_Cell
- removed C5: C_Small, symbol Device:C_Small
- removed D1: D_ALT, symbol Device:D_ALT
- removed Q3: A0448, Package_TO_SOT_SMD:TDSON-8-1, symbol Transistor_FET:CSD16342Q5A
- removed TP1: 12V+, symbol Connector:TestPoint
- removed TP2: OUTPUT, symbol Connector:TestPoint
- removed TP3: 12V-, symbol Connector:TestPoint
- added C10: 10uf, symbol Device:C_Small
- added C11: .1uf, symbol Device:C_Small
- added C5, C6, C7: ?uf, symbol Device:CP1_Small
- added C8, C9: 1uf, symbol Device:C_Small
- added D1: D_Zener, symbol Device:D_Zener
- added R10, R11, R12, R13, R8, R9: ?k, symbol Device:R_Small
- added R?: 10k, symbol Device:R_Small
- added SW?: Momentary, symbol Switch:SW_Push_Open_Dual_x2
- added U1: MC33063AD, Package_SO:SOIC-8_3.9x4.9mm_P1.27mm, symbol Regulator_Switching:MC33063AD
- added U2: NCP718A, Footprints:SON65P200X200X80-7N, symbol Regulator_Linear:AP2204K-ADJ
- added U3: ATtiny20-CCU, Package_BGA:UFBGA-15_3.0x3.0mm_Layout4x4_P0.65mm, symbol MCU_Microchip_ATtiny:ATtiny20-CCU
- L1: value L_Core_Iron -> 10uH
Connections:
- net labels added: +12V, +BATT, MIC_IN, MODE
- wire segments 34 -> 71
Other:
- note added: "Button\n"
- note added: "Design Requirements:\n\nC9 close to U2\nC10 & C11 close to U3\nFeedback line on U1 as short as possible"
- note added: "Microphone Pre Amplifier"
- note added: "Power Delivery\n"
- note added: "Temperature Sensing"
- note added: "Voltage Sensing\n"
- moved on the sheet: C1, C2, C3, C4, MK1, Q1, Q2, R1, R2, R3, R4, R5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

Commit message: schematic
Parts:
- added R? (x4): ?k, symbol Device:R_Small
- added TH?: Thermistor, symbol Device:Thermistor
Connections:
- net +12V: now also C7.1, C8.1, D1.1 (K), R11.1, U2.1 (VIN), U2.3 (EN)
- net +BATT: now also R?.1, TH?.1
- net GND: now also R?.1, R?.2
- new net: R?.1, R?.2, R?.2
- new net Pack_Sense: R?.1
- new net Temp_Sense: R?.2, TH?.2
Other:
- moved on the sheet: C1, C2, C3, C4, MK1, Q1, Q2, R1, R2, R3, R4, R5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

Commit message: schematic done. just calculate values now
Parts:
- added Q3: A04484, Package_TO_SOT_SMD:TDSON-8-1, symbol Transistor_FET:CSD16342Q5A
- added R19: ?k, symbol Device:R_Small
- added R20: 10k, symbol Device:R_Small
- added TP1: LED-, symbol Connector:TestPoint
- added TP2: LED+, symbol Connector:TestPoint
- U3: symbol MCU_Microchip_ATtiny:ATtiny20-CCU -> Main-Board-rescue:ATtiny20-CCU-MCU_Microchip_ATtiny
- gave numbers to parts that had none: 7
Connections:
- net +12V: now also TP2.1
- net GND: now also Q3.1 (S), Q3.2 (S), Q3.3 (S), R19.1
- new net: Q3.4 (G), R20.1
- new net: Q3.5 (D), TP1.1
- new net LED: R19.2, R20.2
Other:
- moved on the sheet: C1, C10, C11, C2, C3, C4, C5, C6, C7, C8, C9, D1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

Commit message: calculated values for schematic
Parts:
- removed C4: 0.1uf, symbol Device:CP1_Small
- C5: value ?uf -> 100uf
- C6: value ?uf -> 320pf
- C7: value ?uf -> 470
- D1: value D_Zener -> 1N5819
- R1: value 10k -> 6.8k
- R10: value ?k -> 180
- R11: value ?k -> 24k
- R18: value ?k -> 10k
- R8: value ?k -> 3k
- R9: value ?k -> 0.08
Changed lines of the file:
@@
 Comment4 ""
 $EndDescr
-Connection ~ 2100 4590
-Wire Wire Line
-	1960 4590 2100 4590
-Connection ~ 2100 4790
-Wire Wire Line
-	2100 4790 1960 4790
-$Comp
-L Device:CP1_Small C4
-U 1 1 5EB56011
-P 1960 4690
-F 0 "C4" H 1810 4730 50  0000 C CNN
-F 1 "0.1uf" H 1780 4650 50  0000 C CNN
-F 2 "" H 1960 4690 50  0001 C CNN
-F 3 "~" H 1960 4690 50  0001 C CNN
-	1    1960 4690
-	1    0    0    -1
-$EndComp
 Wire Wire Line
 	2100 3640 2100 3900
@@
 P 950 4150
 F 0 "R1" H 1009 4196 50  0000 L CNN
-F 1 "10k" H 1009 4105 50  0000 L CNN
+F 1 "6.8k" H 1009 4105 50  0000 L CNN
 F 2 "" H 950 4150 50  0001 C CNN
 F 3 "~" H 950 4150 50  0001 C CNN
@@
 $EndComp
 $Comp
-L Device:Q_NPN_BEC Q1
-U 1 1 5EB26D32
-P 2000 4390
-F 0 "Q1" H 2191 4436 50  0000 L CNN
-F 1 "NPN" H 2191 4345 50  0000 L CNN
-F 2 "" H 2200 4490 50  0001 C CNN
-F 3 "~" H 2000 4390 50  0001 C CNN
-	1    2000 4390
-	1    0    0    -1
-$EndComp
-$Comp
 L Device:CP1_Small C2
 U 1 1 5EB248DC
@@
 P 950 2690
 F 0 "C6" H 800 2730 50  0000 C CNN
-F 1 "?uf" H 770 2650 50  0000 C CNN
+F 1 "320pf" H 770 2650 50  0000 C CNN
 F 2 "" H 950 2690 50  0001 C CNN
 F 3 "~" H 950 2690 50  0001 C CNN
@@
 P 2550 2890
 F 0 "C7" H 2400 2930 50  0000 C CNN
-F 1 "?uf" H 2370 2850 50  0000 C CNN
+F 1 "470" H 2370 2850 50  0000 C CNN
 F 2 "" H 2550 2890 50  0001 C CNN
 F 3 "~" H 2550 2890 50  0001 C CNN
@@
 P 1850 2890
 F 0 "R8" H 1910 2920 50  0000 L CNN
-F 1 "?k" H 1900 2850 50  0000 L CNN
+F 1 "3k" H 1900 2850 50  0000 L CNN
 F 2 "" H 1850 2890 50  0001 C CNN
 F 3 "~" H 1850 2890 50  0001 C CNN
@@
 P 2210 2790
 F 0 "R11" V 2080 2730 50  0000 L CNN
-F 1 "?k" V 2140 2740 50  0000 L CNN
+F 1 "24k" V 2140 2740 50  0000 L CNN
 F 2 "" H 2210 2790 50  0001 C CNN
 F 3 "~" H 2210 2790 50  0001 C CNN
 	1    2210 2790
 	0    1    1    0
-$EndComp
-$Comp
-L Device:CP1_Small C5
-U 1 1 5EC0C8BD
-P 940 2290
-F 0 "C5" H 790 2330 50  0000 C CNN
-F 1 "?uf" H 760 2250 50  0000 C CNN
-F 2 "" H 940 2290 50  0001 C CNN
-F 3 "~" H 940 2290 50  0001 C CNN
-	1    940  2290
-	1    0    0    -1
 $EndComp
 Wire Wire Line
@@
 P 2060 2290
 F 0 "R10" V 2020 2070 50  0000 L CNN
-F 1 "?k" V 2100 2090 50  0000 L CNN
+F 1 "180" V 2100 2060 50  0000 L CNN
 F 2 "" H 2060 2290 50  0001 C CNN
 F 3 "~" H 2060 2290 50  0001 C CNN
@@
 Wire Wire Line
 	1850 2290 1960 2290
-$Comp
-L Device:R_Small R9
-U 1 1 5EBF339E
-P 2060 2190
-F 0 "R9" V 2180 2140 50  0000 L CNN
-F 1 "?k" V 2119 2145 50  0000 L CNN
-F 2 "" H 2060 2190 50  0001 C CNN
-F 3 "~" H 2060 2190 50  0001 C CNN
-	1    2060 2190
-	0    -1   -1   0
-$EndComp
 Wire Wire Line
 	1850 2190 1960 2190
@@
 P 2550 2540
 F 0 "D1" V 2596 2461 50  0000 R CNN
-F 1 "D_Zener" V 2505 2461 50  0000 R CNN
+F 1 "1N5819" V 2505 2461 50  0000 R CNN
 F 2 "" H 2550 2540 50  0001 C CNN
 F 3 "~" H 2550 2540 50  0001 C CNN
@@
 $EndComp
 $Comp
-L Device:R_Small R15
-U 1 1 5EBF785D
-P 2230 5660
-F 0 "R15" H 2290 5690 50  0000 L CNN
-F 1 "?k" H 2280 5620 50  0000 L CNN
-F 2 "" H 2230 5660 50  0001 C CNN
-F 3 "~" H 2230 5660 50  0001 C CNN
-	1    2230 5660
-	1    0    0    -1
-$EndComp
-$Comp
 L power:+BATT #PWR020
 U 1 1 5EBF7B66
@@
 F 3 "" H 2230 5490 50  0001 C CNN
 	1    2230 5490
-	1    0    0    -1
-$EndComp
-$Comp
-L Device:R_Small R16
-U 1 1 5EBF86E0
-P 2230 5860
-F 0 "R16" H 2290 5890 50  0000 L CNN
-F 1 "?k" H 2280 5820 50  0000 L CNN
-F 2 "" H 2230 5860 50  0001 C CNN
-F 3 "~" H 2230 5860 50  0001 C CNN
-	1    2230 5860
-	1    0    0    -1
-$EndComp
-$Comp
-L power:GND #PWR021
-U 1 1 5EBF8995
-P 2230 5960
-F 0 "#PWR021" H 2230 5710 50  0001 C CNN
-F 1 "GND" H 2235 5787 50  0000 C CNN
-F 2 "" H 2230 5960 50  0001 C CNN
-F 3 "" H 2230 5960 50  0001 C CNN
-	1    2230 5960
 	1    0    0    -1
 $EndComp
@@
 Wire Wire Line
 	2460 5760 2230 5760
-Connection ~ 2230 5760
 Text Label 3140 5760 2    50   ~ 0
 Pack_Sense
@@
 P 3820 5770
 F 0 "R18" V 3680 5710 50  0000 L CNN
-F 1 "?k" V 3740 5700 50  0000 L CNN
+F 1 "10k" V 3740 5700 50  0000 L CNN
 F 2 "" H 3820 5770 50  0001 C CNN
 F 3 "~" H 3820 5770 50  0001 C CNN
@@
 Text Label 5160 5440 2    50   ~ 0
 LED
+$Comp
+L Device:Q_NPN_BEC Q1
+U 1 1 5EB26D32
+P 2000 4390
+F 0 "Q1" H 2191 4436 50  0000 L CNN
+F 1 "NPN" H 2191 4345 50  0000 L CNN
+F 2 "" H 2200 4490 50  0001 C CNN
+F 3 "~" H 2000 4390 50  0001 C CNN
+	1    2000 4390
+	1    0    0    -1
+$EndComp
+$Comp
+L Device:R_Small R9
+U 1 1 5EBF339E
+P 2060 2190
+F 0 "R9" V 2180 2140 50  0000 L CNN
+F 1 "0.08" V 2120 2100 50  0000 L CNN
+F 2 "" H 2060 2190 50  0001 C CNN
+F 3 "~" H 2060 2190 50  0001 C CNN
+	1    2060 2190
+	0    -1   -1   0
+$EndComp
+Text Label 2600 3010 0    50   ~ 0
+Test_This!
+$Comp
+L Device:CP1_Small C5
+U 1 1 5EC0C8BD
+P 940 2290
+F 0 "C5" H 790 2330 50  0000 C CNN
+F 1 "100uf" H 760 2250 50  0000 C CNN
+F 2 "" H 940 2290 50  0001 C CNN
+F 3 "~" H 940 2290 50  0001 C CNN
+	1    940  2290
+	1    0    0    -1
+$EndComp
+$Comp
+L power:GND #PWR021
+U 1 1 5EBF8995
+P 2230 5960
+F 0 "#PWR021" H 2230 5710 50  0001 C CNN
+F 1 "GND" H 2235 5787 50  0000 C CNN
+F 2 "" H 2230 5960 50  0001 C CNN
+F 3 "" H 2230 5960 50  0001 C CNN
+	1    2230 5960
+	1    0    0    -1
+$EndComp
+$Comp
+L Device:R_Small R16
+U 1 1 5EBF86E0
+P 2230 5860
+F 0 "R16" H 2290 5890 50  0000 L CNN
+F 1 "?k" H 2280 5820 50  0000 L CNN
+F 2 "" H 2230 5860 50  0001 C CNN
+F 3 "~" H 2230 5860 50  0001 C CNN
+	1    2230 5860
+	1    0    0    -1
+$EndComp
+Connection ~ 2230 5760
+$Comp
+L Device:R_Small R15
+U 1 1 5EBF785D
+P 2230 5660
+F 0 "R15" H 2290 5690 50  0000 L CNN
+F 1 "?k" H 2280 5620 50  0000 L CNN
+F 2 "" H 2230 5660 50  0001 C CNN
+F 3 "~" H 2230 5660 50  0001 C CNN
+	1    2230 5660
+	1    0    0    -1
+$EndComp
 $EndSCHEMATC
