File: Hardware/Main Board/_autosave-Main Board.kicad_pcb (KiCad board)
At the start: 2 copper layers, 58 parts, among them Q1 MMBT3904-TP, Q2 MMBT3904-TP, Q3 A04484, SW1 Momentary, U1 MT3608, U2 NCP718A, U3 ATtiny1614

Commit message: Added base code for take 3 of beat detection. We got thisgit add .!
Parts:
- moved R16 76.1 mm to (94.2, 76.5)
- moved R15 73.0 mm to (94.2, 79.5)
- moved C4 66.3 mm to (91.2, 94.2)
- moved R14 63.1 mm to (110.5, 78.7)
- moved R13 61.7 mm to (115.8, 69.2)
- moved R12 60.6 mm to (116.6, 66.3)
- moved C9 53.0 mm to (107.4, 83.8)
- moved R20 51.1 mm to (119.9, 75.7)
- moved R18 48.9 mm to (122.7, 83.8)
- moved FB1 46.5 mm to (103.4, 88.6)
- moved C11 44.0 mm to (120.1, 87.9)
- moved C10 41.8 mm to (118.4, 90.4)
- moved R19 39.4 mm to (132.3, 82.0)
- moved R17 36.7 mm to (131.6, 86.6)
- moved R8 29.6 mm to (131.1, 90.7)
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